Commit message: Stable Apriltag and RViz

File: src/master_pkg/description/master.urdf (robot description, URDF)
Before this commit: robot nav_robot, 3 links, 2 joints
Links:
- removed link camera_link
- removed link imu_link
- added link camera
- added link imu
Joints:
- joint base_to_camera: child camera_link -> camera; origin xyz=0.1 0.0 0.2 rpy=0 0 0 -> xyz=0.1 0.0 0.2 rpy=-1.570796327 0 -1.570796327
- joint base_to_imu: child imu_link -> imu
